File: PCB/A500KB.kicad_pcb (KiCad board)
At the start: 2 copper layers, 447.8 x 139.2 mm, 227 parts, among them J1 Conn_01x31, J2 USB_B_Micro, J3 Conn_02x03_Odd_Even, J4 Conn_01x08_Male, J5 Conn_01x02, Q1 MMBT3904, U1 IS32FL3237_DS, U2 AT90USB1287-AU, Y2 16 MHz

Commit message: V0.3: improvements for CherryMX builds and fitment - plate design for CherryMX PCB mounted stabilizers   (see PCB/A500KBPlate_Gerber_V2D.zip for Costar variant) - PCB modifications for better fitment in A1200.net cases - PCB modification for additional Caps LED option (MX compatible) - 3D Printed part updates - Build notes readme in PCB/
Parts:
- added D69: RGBCAPS, MXMitsumi:LED_Cree-PLCC4_3.2x2.8mm_CCW, F.Cu at (59.3, 317.9)
- added H22: MountingHole, MountingHole:MountingHole_2.5mm, F.Cu at (445.4, 257.3)
- added H23: MountingHole, MountingHole:MountingHole_2.5mm, F.Cu at (465.4, 238.1)
- added J6: Conn_01x04_Male, Connector_PinHeader_2.54mm:PinHeader_1x04_P2.54mm_Vertical, F.Cu at (403.1, 249.3)
- C15: value 47uF SVP 47/10 -> N/A
- C16: value 47 uF SVP 47/10 -> N/A
- R11: value 10k -> N/A
- moved H6 41.1 mm to (27.9, 262.2)
- moved D13 4.72 mm to (172.6, 336.2)
- moved D7 1.05 mm to (460.1, 251.4)
- moved D53 1.04 mm to (460.1, 243.4)
- moved H2 1.03 mm to (448.1, 251.4)
- moved D4 1.03 mm to (455.9, 251.3)
- moved H1 1.00 mm to (463.9, 251.4)
- moved H3 1.00 mm to (448.1, 243.4)
- moved H4 1.00 mm to (463.9, 243.4)
- moved D52 0.99 mm to (456.1, 243.4)
- moved D6 0.98 mm to (456.1, 251.4)
- moved D5 0.98 mm to (452.1, 251.4)
- moved D51 0.97 mm to (452.1, 243.4)
- moved D3 0.97 mm to (456.0, 243.4)
- moved MX1 0.05 mm to (35.5, 246.2)
Routing:
- net +5V: track 840.7 -> 888.5 mm, vias 8 -> 12
- net /CAPSB: track 447.9 -> 488.3 mm
- net /CAPSG: track 448.0 -> 484.8 mm
- net /CAPSR: track 454.4 -> 483.4 mm
- net /SDA: track 109.4 -> 115.2 mm
- net GND: track 899.2 -> 904.6 mm, vias 161 -> 170
- net /SCL: track 112.0 -> 116.8 mm
- net /X6=3: track 450.5 -> 446.0 mm
- net /FLED: track 52.8 -> 48.7 mm
- net /Y9=20: track 721.8 -> 718.7 mm
- net /F1G: track 19.8 -> 17.1 mm
- net /F2G: track 26.9 -> 24.3 mm
- net /F1B: track 19.0 -> 16.5 mm
- net Net-(D13-Pad2): track 22.9 -> 25.3 mm, vias 0 -> 1
- net /F3G: track 30.3 -> 28.1 mm
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Other:
- outline, holes or cut-outs redrawn
- board text added: "A500KB for Mitsumi or Cherry switches Rev.3b © 2021-24 Henryk Richter"
- board text added: "I2C reserved"
- board text added: "MX CAPSLED"
- board text added: "SCL"
- board text added: "SDA"
- board text removed: "A500KB for Mitsumi or Cherry switches Rev.2 © 2021-22 Henryk Richter"
