File: PCB/A500KBPlate.kicad_pcb (KiCad board)
At the start: 2 copper layers, 448.3 x 124.5 mm, 114 parts, among them J1 Conn_01x04

Commit message: Some more adjustments to Footprints, updated doc
Parts:
- added H3: MountingHole, MountingHole:MountingHole_4.3mm_M4, F.Cu at (49.8, 246.2)
- added H4: MountingHole, MountingHole:MountingHole_4.3mm_M4, F.Cu at (392.4, 293.9)
- moved D12 7.46 mm to (384.8, 292.4)
Routing:
- net Net-(D11-Pad6): track 37.1 -> 28.5 mm
- net Net-(D11-Pad5): track 32.2 -> 24.5 mm
- net Net-(D12-Pad5): track 34.6 -> 38.4 mm
- net /GND: track 624.4 -> 622.0 mm, vias 32 -> 33
- net Net-(D12-Pad6): track 35.6 -> 37.9 mm
- net /+5V: track 590.1 -> 588.3 mm

Commit message: finalized V2 design, LED defaults include IN4 now
Routing:
- net Net-(D8-Pad6): track 301.4 -> 315.5 mm, vias 2 -> 0
- net Net-(D8-Pad5): track 300.8 -> 310.9 mm, vias 2 -> 0
- net Net-(D11-Pad5): track 24.5 -> 30.4 mm
- net Net-(D11-Pad6): track 28.5 -> 26.6 mm, vias 2 -> 0
- net /GND: track 622.0 -> 622.3 mm, vias 33 -> 0
- removed copper zone on B.Cu, net /GND
Other:
- net class Default: via_dia 0.8 -> 1
- rule via_min_size: 0.4 -> 1
- board text removed: "+5V"
- board text removed: "CLK"
- board text removed: "DAT"
- board text removed: "GND"

Commit message: V0.3: improvements for CherryMX builds and fitment - plate design for CherryMX PCB mounted stabilizers   (see PCB/A500KBPlate_Gerber_V2D.zip for Costar variant) - PCB modifications for better fitment in A1200.net cases - PCB modification for additional Caps LED option (MX compatible) - 3D Printed part updates - Build notes readme in PCB/
Parts:
- added REF**: baxlogo, Bax:baxlogo, F.Cu at (334.0, 357.1)
- J1: footprint Connector_PinHeader_2.54mm:PinHeader_1x04_P2.54mm_Horizontal -> Connector_PinHeader_2.54mm:PinHeader_1x04_P2.54mm_Vertical_SMD_Pin1Left
- MX3, MX83: footprint MXMitsumi:MXMitsumi-2U-PlateCutout -> MXMitsumi:MXMitsumi-2U-PlateCutout_Cherry
- MX33: footprint MXMitsumi:MXMitsumi-9U-PlateCutout -> MXMitsumi:MXMitsumi-9U-PlateCutout_Cherry
- MX68: footprint MXMitsumi:MXMitsumi-2.75U-PlateCutout -> MXMitsumi:MXMitsumi-2.75U-PlateCutout_Cherry
- MX71: footprint MXMitsumi:MXMitsumi-ISO-PlateCutout -> MXMitsumi:MXMitsumi-ISO-PlateCutout_Cherry
- MX96: footprint MXMitsumi:MXMitsumi-2U-VerticalStabilizers-PlateCutout -> MXMitsumi:MXMitsumi-2U-VerticalStabilizers-PlateCutout_Cherry
- moved J1 5.24 mm to (297.0, 260.5)
- moved MX1 0.05 mm to (35.5, 246.2)
- turned MX33 to 180 degrees
- turned MX83 to 180 degrees
- turned MX96 to 180 degrees
Connections:
- D15 pad 5: Net-(D15-Pad5) -> (no net)
- D15 pad 6: Net-(D15-Pad6) -> (no net)
Routing:
- net /DAT: track 19.4 -> 16.1 mm
- net /+5V: track 588.3 -> 586.3 mm
- net /CLK: track 19.8 -> 18.4 mm
Other:
- board size 448.3 x 124.5 mm -> 448.3 x 126.5 mm
- board text added: "+5V"
- board text added: "A500KB Plate for Cherry switches Rev.3b © 2021-24 Henryk Richter"
- board text added: "CLK"
- board text added: "DAT"
- board text added: "GND"

Commit message: V4: optional LED strip on full PCB
Parts:
- removed D1, D10, D11, D12, D13, D14, D15, D2, D3, D4, D5, D6, D7, D8, D9: APA102, LED_SMD:LED_RGB_5050-6
- removed J1: Conn_01x04, Connector_PinHeader_2.54mm:PinHeader_1x04_P2.54mm_Vertical_SMD_Pin1Left
- removed REF**: baxlogo, Bax:baxlogo
- added LEDC1: ~, LED_Cutout_Lib:LED_Cutout, F.Cu at (35.7, 260.2)
- added LEDC10: ~, LED_Cutout_Lib:LED_Cutout, F.Cu at (326.0, 274.7)
- added LEDC11: ~, LED_Cutout_Lib:LED_Cutout, F.Cu at (359.1, 293.9)
- added LEDC12: ~, LED_Cutout_Lib:LED_Cutout, F.Cu at (392.5, 274.7)
- added LEDC13: ~, LED_Cutout_Lib:LED_Cutout, F.Cu at (392.5, 331.9)
- added LEDC14: ~, LED_Cutout_Lib:LED_Cutout, F.Cu at (359.2, 346.0)
- added LEDC15: ~, LED_Cutout_Lib:LED_Cutout, F.Cu at (326.0, 331.9)
- added LEDC2: ~, LED_Cutout_Lib:LED_Cutout, F.Cu at (67.5, 260.2)
- added LEDC3: ~, LED_Cutout_Lib:LED_Cutout, F.Cu at (99.3, 260.2)
- added LEDC4: ~, LED_Cutout_Lib:LED_Cutout, F.Cu at (131.1, 260.2)
- added LEDC5: ~, LED_Cutout_Lib:LED_Cutout, F.Cu at (162.9, 260.2)
- added LEDC6: ~, LED_Cutout_Lib:LED_Cutout, F.Cu at (194.6, 260.2)
- added LEDC7: ~, LED_Cutout_Lib:LED_Cutout, F.Cu at (226.4, 260.2)
- added LEDC8: ~, LED_Cutout_Lib:LED_Cutout, F.Cu at (258.2, 260.2)
- added LEDC9: ~, LED_Cutout_Lib:LED_Cutout, F.Cu at (290.0, 260.2)
- added baxlogo1: Baxlogo, Bax:baxlogo, F.Cu at (334.0, 357.2)
- MX1, MX10, MX11, MX14, MX15, MX16, MX17, MX19, MX20, MX21, MX22, MX24, MX25, MX26, MX27, MX29, MX30, MX31, MX32, MX35, MX36, MX37, MX38, MX40, MX41, MX42, MX43, MX45, MX46, MX47, MX48, MX50, MX51, MX52, MX53, MX55, MX56, MX57, MX58, MX60, MX61, MX62, MX63, MX65, MX66, MX67, MX69, MX70, MX72, MX74, MX75, MX76, MX78, MX79, MX8, MX80, MX81, MX82, MX84, MX85, MX86, MX87, MX88, MX89, MX9, MX90, MX91, MX92, MX93, MX94, MX95: footprint MXMitsumi:MXMitsumi-1U-PlateCutout -> MXMitsumi:MXMitsumi-1U-PlateCutout_Square
- MX12, MX13, MX18, MX23, MX28, MX34, MX39, MX4, MX44, MX49, MX54, MX59, MX6, MX64, MX7: footprint MXMitsumi:MXMitsumi-1.25U-PlateCutout -> MXMitsumi:MXMitsumi-1.25U-PlateCutout_Square
Routing:
- net /GND: track 622.7 -> 0.00 mm
- net /+5V: track 586.3 -> 0.00 mm
- net Net-(D8-Pad6): track 315.5 -> 0.00 mm
- net Net-(D8-Pad5): track 311.4 -> 0.00 mm
- net Net-(D13-Pad6): track 49.6 -> 0.00 mm
- net Net-(D13-Pad5): track 48.8 -> 0.00 mm
- net Net-(D14-Pad6): track 46.8 -> 0.00 mm
- net Net-(D14-Pad5): track 45.0 -> 0.00 mm
- net Net-(D12-Pad5): track 38.4 -> 0.00 mm
- net Net-(D12-Pad6): track 37.9 -> 0.00 mm
- net Net-(D10-Pad5): track 36.7 -> 0.00 mm
- net Net-(D5-Pad6): track 34.4 -> 0.00 mm
- net Net-(D5-Pad5): track 33.4 -> 0.00 mm
- net Net-(D7-Pad6): track 32.9 -> 0.00 mm
- net Net-(D7-Pad5): track 31.9 -> 0.00 mm
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- added copper zone on F.Cu, net (none)
- removed copper zone on F.Cu, net /GND
Other:
- net class Default removed
- board text removed: "+5V"
- board text removed: "CLK"
- board text removed: "DAT"
- board text removed: "GND"

Commit message: shifted A500KB connectors down on the PCB by 9mm This change allows angled connectors in conjunction with Dupont plugs for connection to the A500 mainboard.
Parts:
- H3, H4: footprint MountingHole:MountingHole_4.3mm_M4 -> MountingHole:MountingHole_4mm
Changed lines of the file:
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@@
 		)
 	)
-	(footprint "MountingHole:MountingHole_4.3mm_M4"
+	(footprint "MountingHole:MountingHole_4mm"
 		(layer "F.Cu")
 		(at 392.45 293.85)
-		(descr "Mounting Hole 4.3mm, no annular, M4")
-		(tags "mounting hole 4.3mm no annular m4")
+		(descr "Mounting Hole 4mm, no annular")
+		(tags "mounting hole 4mm no annular")
 		(property "Reference" "H4"
-			(at 0 -5.3 0)
+			(at 0 -5 0)
 			(layer "F.SilkS")
 			(effects
@@
 		)
 		(property "Value" "MountingHole"
-			(at 0 5.3 0)
-			(layer "F.Fab")
-			(effects
-				(font
-					(size 1 1)
-					(thickness 0.15)
-				)
-			)
-		)
-		(property "Footprint" "MountingHole:MountingHole_4.3mm_M4"
-			(at 0 0 0)
+			(at 0 5 0)
+			(layer "F.Fab")
+			(effects
+				(font
+					(size 1 1)
+					(thickness 0.15)
+				)
+			)
+		)
+		(property "Footprint" "MountingHole:MountingHole_4mm"
+			(at 0 0 0)
+			(unlocked yes)
 			(layer "F.Fab")
 			(hide yes)
@@
 		(property "Datasheet" ""
 			(at 0 0 0)
+			(unlocked yes)
 			(layer "F.Fab")
 			(hide yes)
@@
 		(property "Description" ""
 			(at 0 0 0)
+			(unlocked yes)
 			(layer "F.Fab")
 			(hide yes)
@@
 		(fp_circle
 			(center 0 0)
-			(end 4.3 0)
+			(end 4 0)
 			(stroke
 				(width 0.15)
@@
 		(fp_circle
 			(center 0 0)
-			(end 4.55 0)
+			(end 4.25 0)
 			(stroke
 				(width 0.05)
@@
 		)
 		(fp_text user "${REFERENCE}"
-			(at 0.3 0 0)
+			(at 0 0 0)
 			(layer "F.Fab")
 			(effects
@@
 		(pad "" np_thru_hole circle
 			(at 0 0)
-			(size 6 6)
-			(drill 6)
-			(layers "F&B.Cu" "*.Mask")
+			(size 4 4)
+			(drill 4)
+			(layers "*.Cu" "*.Mask")
 		)
 	)
-	(footprint "MountingHole:MountingHole_4.3mm_M4"
+	(footprint "MountingHole:MountingHole_4mm"
 		(layer "F.Cu")
 		(at 49.75 246.15)
-		(descr "Mounting Hole 4.3mm, no annular, M4")
-		(tags "mounting hole 4.3mm no annular m4")
+		(descr "Mounting Hole 4mm, no annular")
+		(tags "mounting hole 4mm no annular")
 		(property "Reference" "H3"
-			(at 0 -5.3 0)
+			(at 0 -5 0)
 			(layer "F.SilkS")
 			(effects
@@
 		)
 		(property "Value" "MountingHole"
-			(at 0 5.3 0)
-			(layer "F.Fab")
-			(effects
-				(font
-					(size 1 1)
-					(thickness 0.15)
-				)
-			)
-		)
-		(property "Footprint" "MountingHole:MountingHole_4.3mm_M4"
-			(at 0 0 0)
+			(at 0 5 0)
+			(layer "F.Fab")
+			(effects
+				(font
+					(size 1 1)
+					(thickness 0.15)
+				)
+			)
+		)
+		(property "Footprint" "MountingHole:MountingHole_4mm"
+			(at 0 0 0)
+			(unlocked yes)
 			(layer "F.Fab")
 			(hide yes)
@@
 		(property "Datasheet" ""
 			(at 0 0 0)
+			(unlocked yes)
 			(layer "F.Fab")
 			(hide yes)
@@
 		(property "Description" ""
 			(at 0 0 0)
+			(unlocked yes)
 			(layer "F.Fab")
 			(hide yes)
@@
 		(fp_circle
 			(center 0 0)
-			(end 4.3 0)
+			(end 4 0)
 			(stroke
 				(width 0.15)
@@
 		(fp_circle
 			(center 0 0)
-			(end 4.55 0)
+			(end 4.25 0)
 			(stroke
 				(width 0.05)
@@
 		)
 		(fp_text user "${REFERENCE}"
-			(at 0 -3.35 0)
+			(at 0 0 0)
 			(layer "F.Fab")
 			(effects
@@
 		(pad "" np_thru_hole circle
 			(at 0 0)
-			(size 6 6)
-			(drill 6)
-			(layers "F&B.Cu" "*.Mask")
+			(size 4 4)
+			(drill 4)
+			(layers "*.Cu" "*.Mask")
 		)
 	)
